Commit message: third

File: box1/src/urdf02_gazebo/urdf/demo07_laser.xacro (robot description, xacro)
@@ -8,4 +8,5 @@
     <xacro:property name="support_x" value="0.0" /> <!-- 支架安装的x坐标 -->
     <xacro:property name="support_y" value="0.0" /> <!-- 支架安装的y坐标 -->
+    <xacro:property name="support_z" value="${base_link_length / 2 + support_length / 2}" /> <!-- 支架安装的z坐标:底盘高度 / 2 + 支架高度 / 2  -->
     <xacro:property name="support_m" value="0.02" /> <!-- 支架质量 -->
     <link name="support">
